File: Miniscope-v4-Wire-Free-KiCad/KiCad/EWL_FlexPC/KiCad/EWL_FlexPC.kicad_pcb (KiCad board)
At the start: 2 copper layers, 14.6 x 20.8 mm, 0 parts

Commit message: Update public repository
- Made copy to a public repository
Other:
- outline, holes or cut-outs redrawn
Changed lines of the file:
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@@
-(kicad_pcb (version 20211014) (generator pcbnew)
+(kicad_pcb (version 20221018) (generator pcbnew)
   (general
     (thickness 1.6)
@@
     (pcbplotparams
       (layerselection 0x00010fc_ffffffff)
+      (plot_on_all_layers_selection 0x0000000_00000000)
       (disableapertmacros false)
       (usegerberextensions false)
@@
       (usegerberadvancedattributes false)
       (creategerberjobfile false)
-      (svguseinch false)
+      (dashed_line_dash_ratio 12.000000)
+      (dashed_line_gap_ratio 3.000000)
       (svgprecision 6)
-      (excludeedgelayer true)
       (plotframeref false)
       (viasonmask false)
@@
   )
   (net 0 "")
-  (gr_arc (start 47.155974 31.03514) (mid 51.567955 27.411272) (end 50.4 33) (layer "F.Cu") (width 0.7))
-  (gr_circle (center 43 37) (end 46.4 37) (layer "F.Cu") (width 0.3) (fill none))
-  (gr_line (start 49.575 45.45) (end 49.6 33.5) (layer "F.Cu") (width 0.3048))
-  (gr_line (start 50.375 45.45) (end 50.4 33) (layer "F.Cu") (width 0.3048))
-  (gr_line (start 47.509016 32.490984) (end 45.5 34.6) (layer "F.Cu") (width 0.3048))
-  (gr_arc (start 49.6 33.5) (mid 48.468995 33.1727) (end 47.509016 32.490984) (layer "F.Cu") (width 0.3048))
-  (gr_poly
-    (pts
-      (xy 50.175 44.775)
-      (xy 50.175 46.55)
-      (xy 50.175 46.65)
-      (xy 50.675 46.65)
-      (xy 50.675 44.775)
-    ) (layer "F.Cu") (width 0.1) (fill solid))
-  (gr_poly
-    (pts
-      (xy 49.275 44.775)
-      (xy 49.275 46.55)
-      (xy 49.275 46.65)
-      (xy 49.775 46.65)
-      (xy 49.775 44.775)
-    ) (layer "F.Cu") (width 0.1) (fill solid))
-  (gr_poly
-    (pts
-      (xy 49.275 44.775)
-      (xy 49.275 46.55)
-      (xy 49.275 46.65)
-      (xy 49.775 46.65)
-      (xy 49.775 44.775)
-    ) (layer "B.Cu") (width 0.1) (fill solid))
-  (gr_poly
-    (pts
-      (xy 50.175 44.775)
-      (xy 50.175 46.55)
-      (xy 50.175 46.65)
-      (xy 50.675 46.65)
-      (xy 50.675 44.775)
-    ) (layer "B.Cu") (width 0.1) (fill solid))
-  (gr_circle (center 50.425 46.05) (end 50.552 46.05) (layer "B.Mask") (width 0.254) (fill none))
-  (gr_circle (center 49.527 46.075) (end 49.654 46.075) (layer "B.Mask") (width 0.254) (fill none))
-  (gr_poly
-    (pts
-      (xy 49.275 44.775)
-      (xy 49.275 46.55)
-      (xy 49.275 46.65)
-      (xy 49.775 46.65)
-      (xy 49.775 44.775)
-    ) (layer "B.Mask") (width 0.1) (fill solid))
-  (gr_poly
-    (pts
-      (xy 50.175 44.775)
-      (xy 50.175 46.55)
-      (xy 50.175 46.65)
-      (xy 50.675 46.65)
-      (xy 50.675 44.775)
-    ) (layer "B.Mask") (width 0.1) (fill solid))
-  (gr_circle (center 50 30) (end 52.925 30) (layer "F.Mask") (width 0.45) (fill none))
-  (gr_circle (center 43 37) (end 46.5 37) (layer "F.Mask") (width 0.5) (fill none))
-  (gr_poly
-    (pts
-      (xy 49.275 44.775)
-      (xy 49.275 46.55)
-      (xy 49.275 46.65)
-      (xy 49.775 46.65)
-      (xy 49.775 44.775)
-    ) (layer "F.Mask") (width 0.1) (fill solid))
-  (gr_poly
-    (pts
-      (xy 50.175 44.775)
-      (xy 50.175 46.55)
-      (xy 50.175 46.65)
-      (xy 50.675 46.65)
-      (xy 50.675 44.775)
-    ) (layer "F.Mask") (width 0.1) (fill solid))
-  (gr_arc (start 49.000001 33.699999) (mid 48.327412 33.448542) (end 47.713529 33.076043) (layer "Edge.Cuts") (width 0.15))
-  (gr_arc (start 45.999999 34.800001) (mid 40.369412 39.630588) (end 45.199999 34.000001) (layer "Edge.Cuts") (width 0.15))
-  (gr_line (start 49 47) (end 51 47) (layer "Edge.Cuts") (width 0.15))
-  (gr_line (start 46.921924 32.283734) (end 45.2 34) (layer "Edge.Cuts") (width 0.15))
-  (gr_line (start 49 47) (end 49 33.7) (layer "Edge.Cuts") (width 0.15))
-  (gr_line (start 47.713529 33.076043) (end 45.999999 34.800001) (layer "Edge.Cuts") (width 0.15))
-  (gr_line (start 51 47) (end 51 33.7) (layer "Edge.Cuts") (width 0.15))
-  (gr_circle (center 50 30) (end 52.5476 30) (layer "Edge.Cuts") (width 0.15) (fill none))
-  (gr_arc (start 46.921924 32.283734) (mid 51.257399 26.379373) (end 50.999999 33.699999) (layer "Edge.Cuts") (width 0.15))
-  (gr_circle (center 43 37) (end 43.1 40.1) (layer "Edge.Cuts") (width 0.15) (fill none))
+  (gr_arc (start 47.155974 31.03514) (mid 51.567955 27.411272) (end 50.4 33)
+    (stroke (width 0.7) (type solid)) (layer "F.Cu"))
+  (gr_circle (center 43 37) (end 46.4 37)
+    (stroke (width 0.3) (type solid)) (fill none) (layer "F.Cu"))
+  (gr_line (start 48.575 45.45) (end 48.6 33.15)
+    (stroke (width 0.3048) (type solid)) (layer "F.Cu"))
+  (gr_line (start 49.375 45.45) (end 49.4 33)
+    (stroke (width 0.3048) (type solid)) (layer "F.Cu"))
+  (gr_line (start 47.509016 32.490984) (end 45.5 34.6)
+    (stroke (width 0.3048) (type solid)) (layer "F.Cu"))
+  (gr_poly
+    (pts
+      (xy 49.18 44.77)
+      (xy 49.18 46.545)
+      (xy 49.18 46.645)
+      (xy 49.68 46.645)
+      (xy 49.68 44.77)
+    )
+    (stroke (width 0.1) (type solid)) (fill solid) (layer "F.Cu"))
+  (gr_poly
+    (pts
+      (xy 48.27 44.775)
+      (xy 48.27 46.55)
+      (xy 48.27 46.65)
+      (xy 48.77 46.65)
+      (xy 48.77 44.775)
+    )
+    (stroke (width 0.1) (type solid)) (fill solid) (layer "F.Cu"))
+  (gr_line (start 47.509016 32.490984) (end 48.6 33.15)
+    (stroke (width 0.3048) (type default)) (layer "F.Cu"))
+  (gr_line (start 49.4 33) (end 50.4 33)
+    (stroke (width 0.3048) (type solid)) (layer "F.Cu"))
+  (gr_poly
+    (pts
+      (xy 48.27 44.775)
+      (xy 48.27 46.55)
+      (xy 48.27 46.65)
+      (xy 48.77 46.65)
+      (xy 48.77 44.775)
+    )
+    (stroke (width 0.1) (type solid)) (fill solid) (layer "B.Cu"))
+  (gr_poly
+    (pts
+      (xy 49.18 44.77)
+      (xy 49.18 46.545)
+      (xy 49.18 46.645)
+      (xy 49.68 46.645)
+      (xy 49.68 44.77)
+    )
+    (stroke (width 0.1) (type solid)) (fill solid) (layer "B.Cu"))
+  (gr_circle (center 49.43 46.045) (end 49.557 46.045)
+    (stroke (width 0.254) (type solid)) (fill none) (layer "B.Mask"))
+  (gr_circle (center 48.522 46.075) (end 48.649 46.075)
+    (stroke (width 0.254) (type solid)) (fill none) (layer "B.Mask"))
+  (gr_poly
+    (pts
+      (xy 48.27 44.775)
+      (xy 48.27 46.55)
+      (xy 48.27 46.65)
+      (xy 48.77 46.65)
+      (xy 48.77 44.775)
+    )
+    (stroke (width 0.1) (type solid)) (fill solid) (layer "B.Mask"))
+  (gr_poly
+    (pts
+      (xy 49.18 44.77)
+      (xy 49.18 46.545)
+      (xy 49.18 46.645)
+      (xy 49.68 46.645)
+      (xy 49.68 44.77)
+    )
+    (stroke (width 0.1) (type solid)) (fill solid) (layer "B.Mask"))
+  (gr_circle (center 50 30) (end 52.925 30)
+    (stroke (width 0.45) (type solid)) (fill none) (layer "F.Mask"))
+  (gr_circle (center 43 37) (end 46.5 37)
+    (stroke (width 0.5) (type solid)) (fill none) (layer "F.Mask"))
+  (gr_poly
+    (pts
+      (xy 48.27 44.775)
+      (xy 48.27 46.55)
+      (xy 48.27 46.65)
+      (xy 48.77 46.65)
+      (xy 48.77 44.775)
+    )
+    (stroke (width 0.1) (type solid)) (fill solid) (layer "F.Mask"))
+  (gr_poly
+    (pts
+      (xy 49.18 44.77)
+      (xy 49.18 46.545)
+      (xy 49.18 46.645)
+      (xy 49.68 46.645)
+      (xy 49.68 44.77)
+    )
+    (stroke (width 0.1) (type solid)) (fill solid) (layer "F.Mask"))
+  (gr_arc (start 45.999999 34.800001) (mid 40.369412 39.630588) (end 45.199999 34.000001)
+    (stroke (width 0.15) (type solid)) (layer "Edge.Cuts"))
+  (gr_line (start 48 47) (end 50 47)
+    (stroke (width 0.15) (type solid)) (layer "Edge.Cuts"))
+  (gr_line (start 46.921924 32.283734) (end 45.2 34)
+    (stroke (width 0.15) (type solid)) (layer "Edge.Cuts"))
+  (gr_line (start 48 47) (end 48 33.36)
+    (stroke (width 0.15) (type solid)) (layer "Edge.Cuts"))
+  (gr_line (start 47.713529 33.076043) (end 45.999999 34.800001)
+    (stroke (width 0.15) (type solid)) (layer "Edge.Cuts"))
+  (gr_line (start 50 47) (end 50 33.7)
+    (stroke (width 0.15) (type solid)) (layer "Edge.Cuts"))
+  (gr_circle (center 50 30) (end 52.5476 30)
+    (stroke (width 0.15) (type solid)) (fill none) (layer "Edge.Cuts"))
+  (gr_arc (start 46.921924 32.283734) (mid 51.257399 26.379373) (end 50.999999 33.699999)
+    (stroke (width 0.15) (type solid)) (layer "Edge.Cuts"))
+  (gr_circle (center 43 37) (end 43.1 40.1)
+    (stroke (width 0.15) (type solid)) (fill none) (layer "Edge.Cuts"))
+  (gr_line (start 50.999999 33.699999) (end 50 33.7)
+    (stroke (width 0.15) (type default)) (layer "Edge.Cuts"))
+  (gr_line (start 47.713529 33.076043) (end 48 33.36)
+    (stroke (width 0.15) (type solid)) (layer "Edge.Cuts"))
   (gr_text "FH19C Series\n\nThickness : 0.2 ± 0.03mm Gold plated" (at 56.375 35.1) (layer "Cmts.User")
     (effects (font (size 1.5 1.5) (thickness 0.3)) (justify left))
   )
-  (via (at 49.525 46.075) (size 0.508) (drill 0.254) (layers "F.Cu" "B.Cu") (net 0))
-  (via (at 50.425317 46.053808) (size 0.508) (drill 0.254) (layers "F.Cu" "B.Cu") (net 0))
+  (via (at 48.52 46.075) (size 0.508) (drill 0.254) (layers "F.Cu" "B.Cu") (net 0))
+  (via (at 49.430317 46.048808) (size 0.508) (drill 0.254) (layers "F.Cu" "B.Cu") (net 0))
+  (group "PAD1" (id 879609b1-cb6b-483e-96e3-92066a36035d)
+    (members
+      00000000-0000-0000-0000-00005d3f581c
+      00000000-0000-0000-0000-00005d3f5825
+      00000000-0000-0000-0000-00005d3f5828
+      00000000-0000-0000-0000-00005d3f5831
+      6aa0c7aa-154b-4cf1-b26b-41c107eb038a
+      a26bc030-7d8a-4b19-aa84-9206cc0de2b0
+    )
+  )
 )
