File: Miniscope-v4-Wire-Free-KiCad/KiCad/Miniscope-v4-Wire-Free/Miniscope-v4-Wire-Free.sch (KiCad schematic (older format))
At the start: 114 parts, among them J1 0475710001, J10 Conn_01x01, J11 Conn_01x01, J12 Conn_01x01, J14 Conn_01x01, J15 Conn_01x01, J16 Conn_01x01, J17 Conn_01x01, J18 Conn_01x01, J19 Conn_01x01, J2 Conn_01x04, J20 Conn_01x01, J21 Conn_01x01, J22 Conn_01x01, J23 Conn_01x01, J24 Conn_01x01, J25 Conn_01x01, J26 Conn_01x01, J27 Conn_01x01, J3 Conn_01x04, J4 Conn_01x01, J5 Conn_01x01, J6 Conn_01x01, J7 Conn_01x01, J8 Conn_01x01, J9 Conn_01x01, Q1 NTK3134NT1G, Q2 MMBT3904LP-7B, SW1 TL3780AF330QG, U1 LTC3554, U2 HV892, U3 LTC3218, U4 MAX13030EETE+BGA, U5 TSOP57438TT1, U6 ATSAMD51J20A-UUT-EFP, U7 NCP163AMX330TBG, U8 NOIP1SN0480A, U9 LMV321IDCKR, Y2 Crystal

Commit message: Fix to the PCB project
- Reverted the project to KiCAD 6 to avoid breaking microvias when moving to KiCAD 7 or 8
- SPI_CS now connected again

To do:

- Remove the asterisk on the microcontroller silk layer
- Add gerbers for the new PCB
- Discuss with Daniel which numbering version to use
- Add back the 3D models
Parts:
- removed R21: 47k5, .Resistor:R_0201_0603Metric_ERJ_L, symbol .Device:R_Small_US
- L1, L5: PN MLZ1608N100LT00 -> (none)
- L2: PN ASMCI-0805-4R7M-T -> (none)
- L3: value BLM18PG471SN1D -> L_Small
- U1: symbol Miniscope-v4-Wire-Free-rescue:LTC3554-.Regulator_Switching -> .Regulator_Switching:LTC3554; Manufacturer_Part_Number LTC3554EUD#PBF -> (none)
- U2: symbol Miniscope-v4-Wire-Free-rescue:HV892-.Driver_ETL -> .Driver_ETL:HV892
- U4: symbol Miniscope-v4-Wire-Free-rescue:MAX13030EETE+BGA-.Logic_Level_Translator -> .Logic_Level_Translator:MAX13030EETE+BGA
- U6: symbol Miniscope-v4-Wire-Free-rescue:ATSAMD51J20A-UUT-EFP-.SAMD51 -> .SAMD51:ATSAMD51J20A-UUT-EFP
Connections:
- net +3V3: no longer U7.3 (nSHDN)
- net VDC: now also U7.3 (nSHDN)
Other:
- note removed: "Added missing 47k5 resistor"
- note removed: "Changed enable to 3V3\n to comply better with \npower on sequence"
Changed lines of the file:
@@
 $EndComp
 $Comp
-L Miniscope-v4-Wire-Free-rescue:HV892-.Driver_ETL U2
+L .Driver_ETL:HV892 U2
 U 1 1 609F1D8D
 P 20600 7100
@@
 	13150 2800 13150 2900
 Connection ~ 13150 2800
+Wire Wire Line
+	12200 2400 12550 2400
 $Comp
 L power:GND #PWR0108
@@
 	12750 5350 13350 5350
 $Comp
-L Miniscope-v4-Wire-Free-rescue:LTC3554-.Regulator_Switching U1
+L .Regulator_Switching:LTC3554 U1
 U 1 1 60C27DE1
 P 2250 3750
@@
 F 2 "Package_DFN_QFN:QFN-20-1EP_3x3mm_P0.4mm_EP1.65x1.65mm" H 2000 4400 50  0001 C CNN
 F 3 "https://www.analog.com/media/en/technical-documentation/data-sheets/355412ff.pdf" H 2000 4400 50  0001 C CNN
-F 4 "LTC3554EUD#PBF" H 2250 3750 50  0001 C CNN "Manufacturer_Part_Number"
 	1    2250 3750
 	1    0    0    -1
@@
 F 2 ".Capacitor:C_0805_2012Metric_L" H 3050 3700 50  0001 C CNN
 F 3 "~" H 3050 3700 50  0001 C CNN
-F 4 "MLZ1608N100LT00" V 3050 3700 50  0001 C CNN "PN"
 	1    3050 3700
 	0    -1   -1   0
@@
 F 2 ".Capacitor:C_0805_2012Metric_L" H 3050 4400 50  0001 C CNN
 F 3 "~" H 3050 4400 50  0001 C CNN
-F 4 "ASMCI-0805-4R7M-T" V 3050 4400 50  0001 C CNN "PN"
 	1    3050 4400
 	0    -1   -1   0
@@
 	1    0    0    -1
 $EndComp
+$Comp
+L power:VDC #PWR0119
+U 1 1 60F6C172
+P 12200 2400
+F 0 "#PWR0119" H 12200 2300 50  0001 C CNN
+F 1 "VDC" H 12300 2600 50  0000 C CNN
+F 2 "" H 12200 2400 50  0001 C CNN
+F 3 "" H 12200 2400 50  0001 C CNN
+	1    12200 2400
+	1    0    0    -1
+$EndComp
 Wire Wire Line
 	20150 6900 19950 6900
@@
 Wire Wire Line
 	12650 2600 12550 2600
+Wire Wire Line
+	12550 2600 12550 2400
+Connection ~ 12550 2400
+Wire Wire Line
+	12550 2400 12650 2400
 $Comp
 L .Device:C_Small C37
 U 1 1 61434016
 P 12200 2500
-F 0 "C37" H 12276 2492 50  0000 L CNN
-F 1 "1uF" H 12264 2404 50  0000 L CNN
+F 0 "C37" H 12300 2550 50  0000 L CNN
+F 1 "1uF" H 12300 2450 50  0000 L CNN
 F 2 ".Capacitor:C_0201_0603Metric_L" H 12200 2500 50  0001 C CNN
 F 3 "~" H 12200 2500 50  0001 C CNN
@@
 	1    0    0    -1
 $EndComp
+Connection ~ 12200 2400
 Wire Wire Line
 	12200 2600 12200 2800
@@
 U 1 1 61FAC951
 P 7000 1975
-F 0 "L3" V 7074 1978 50  0000 C CNN
-F 1 "BLM18PG471SN1D" V 6929 1986 50  0000 C CNN
+F 0 "L3" V 7200 1975 50  0000 C CNN
+F 1 "L_Small" V 7100 1975 50  0000 C CNN
 F 2 ".Inductor:L_0603_1608Metric_L" H 7000 1975 50  0001 C CNN
 F 3 "~" H 7000 1975 50  0001 C CNN
@@
 PYTHON480
 $Comp
-L Miniscope-v4-Wire-Free-rescue:MAX13030EETE+BGA-.Logic_Level_Translator U4
+L .Logic_Level_Translator:MAX13030EETE+BGA U4
 U 1 1 62728104
 P 18600 12500
@@
 $EndComp
 $Comp
-L Miniscope-v4-Wire-Free-rescue:ATSAMD51J20A-UUT-EFP-.SAMD51 U6
+L .SAMD51:ATSAMD51J20A-UUT-EFP U6
 U 1 1 60A91709
 P 7125 7175
@@
 $EndComp
 $Comp
-L Miniscope-v4-Wire-Free-rescue:ATSAMD51J20A-UUT-EFP-.SAMD51 U6
+L .SAMD51:ATSAMD51J20A-UUT-EFP U6
 U 2 1 60A93C14
 P 7375 3675
@@
 F 2 ".Capacitor:C_0805_2012Metric_L" H 7025 4475 50  0001 C CNN
 F 3 "~" H 7025 4475 50  0001 C CNN
-F 4 "MLZ1608N100LT00" V 7025 4475 50  0001 C CNN "PN"
 	1    7025 4475
 	0    -1   -1   0
@@
 Wire Wire Line
 	6525 7975 7125 7975
-$Comp
-L .Device:R_Small_US R21
-U 1 1 6209E562
-P 13171 7800
-F 0 "R21" V 12971 7850 50  0000 R CNN
-F 1 "47k5" V 13071 7900 50  0000 R CNN
-F 2 ".Resistor:R_0201_0603Metric_ERJ_L" H 13171 7800 50  0001 C CNN
-F 3 "~" H 13171 7800 50  0001 C CNN
-	1    13171 7800
-	1    0    0    -1
-$EndComp
-Wire Wire Line
-	13350 7600 13171 7600
-Wire Wire Line
-	13171 7600 13171 7700
-Wire Wire Line
-	13171 7900 13171 7973
-$Comp
-L power:GND #PWR012
-U 1 1 62193C20
-P 13171 7973
-F 0 "#PWR012" H 13171 7723 50  0001 C CNN
-F 1 "GND" H 13221 7773 50  0000 C CNN
-F 2 "" H 13171 7973 50  0001 C CNN
-F 3 "" H 13171 7973 50  0001 C CNN
-	1    13171 7973
-	1    0    0    -1
-$EndComp
-Connection ~ 12200 2400
-$Comp
-L power:VDC #PWR0119
-U 1 1 60F6C172
-P 12200 2400
-F 0 "#PWR0119" H 12200 2300 50  0001 C CNN
-F 1 "VDC" H 12300 2600 50  0000 C CNN
-F 2 "" H 12200 2400 50  0001 C CNN
-F 3 "" H 12200 2400 50  0001 C CNN
-	1    12200 2400
-	1    0    0    -1
-$EndComp
-Wire Wire Line
-	12200 2400 12650 2400
-$Comp
-L power:+3.3V #PWR01
-U 1 1 62297A3E
-P 12550 2600
-F 0 "#PWR01" H 12550 2450 50  0001 C CNN
-F 1 "+3.3V" H 12534 2740 50  0000 C CNN
-F 2 "" H 12550 2600 50  0001 C CNN
-F 3 "" H 12550 2600 50  0001 C CNN
-	1    12550 2600
-	1    0    0    -1
-$EndComp
-Text Notes 12106 3119 0    50   ~ 0
-Changed enable to 3V3\n to comply better with \npower on sequence
-Text Notes 12117 8303 0    50   ~ 0
-Added missing 47k5 resistor
 $EndSCHEMATC
